Commit message: Add the camera to the Robot

File: rosbots_description/urdf/rosbots.gazebo.xacro (robot description, xacro)
@@ -21,3 +21,35 @@
     </plugin>
   </gazebo>
+<!-- Edit rosbots.gazebo.xacro to add the camera behavior (like take image or record video) to the link, see step 6. Adding the Camera to the Robot -->
+  <gazebo reference="camera_link">
+    <sensor type="camera" name="camera1">
+      <update_rate>30.0</update_rate>
+      <camera name="head">
+        <horizontal_fov>1.04</horizontal_fov>
+        <image>
+          <width>320</width>
+          <height>240</height>
+          <format>R8G8B8</format>
+        </image>
+        <clip>
+          <near>0.1</near>
+          <far>50</far>
+        </clip>
+      </camera>
+      <plugin name="camera_controller" filename="libgazebo_ros_camera.so">
+        <alwaysOn>true</alwaysOn>
+        <updateRate>0</updateRate>
+        <cameraName>camera1</cameraName>
+        <imageTopicName>image_raw</imageTopicName>
+        <cameraInfoTopicName>camera_info</cameraInfoTopicName>
+        <frameName>camera</frameName>
+        <hackBaseline>0.07</hackBaseline>
+        <distortionK1>0.0</distortionK1>
+        <distortionK2>0.0</distortionK2>
+        <distortionK3>0.0</distortionK3>
+        <distortionT1>0.0</distortionT1>
+        <distortionT2>0.0</distortionT2>
+      </plugin>
+    </sensor>
+  </gazebo>
 </robot>

File: rosbots_description/urdf/rosbots.xacro (robot description, xacro)
@@ -1,5 +1,5 @@
 <?xml version="1.0" encoding="utf-8"?>
 <robot name="rosbots" xmlns:xacro="http://www.ros.org/wiki/xacro">
-<!-- tag xacro:include di tambahkan, cek pada step ke 4. Using the XACRO Macros -->
+<!-- tag xacro:include di tambahkan, cek pada step ke 5. Using the XACRO Macros -->
 <xacro:include filename="$(find rosbots_description)/urdf/rosbots.gazebo.xacro" />
     <link name="base_footprint"/>
@@ -385,5 +385,5 @@
       </collision>
     </link>
-    <!-- tag gazebo di nonaktifkan, cek pada step ke 4. Using the XACRO Macros -->
+    <!-- tag gazebo di nonaktifkan, cek pada step ke 5. Using the XACRO Macros -->
     <!-- <gazebo>
         <plugin name="differential_drive_controller" filename="libgazebo_ros_diff_drive.so">
@@ -406,3 +406,24 @@
         </plugin>
     </gazebo> -->
+    <!-- tag camera ditambahkan, cek pada step ke 6. Adding the Camera to the Robot -->
+    <joint name="camera_joint" type="fixed">
+        <origin xyz="0.49 -0.03 0.75" rpy="0 0.21 0" />
+        <parent link="base_link"/>
+        <child link="camera_link" />
+    </joint>
+    <link name="camera_link">
+        <visual>
+            <geometry>
+            <mesh filename="package://duckietown_description/meshes/camera.dae" scale="4.0 4.0 4.0"/>
+            </geometry>
+            <origin xyz="0.0 0 0" rpy="0 0 0"/>
+        </visual>
+        <collision>
+            <geometry>
+            <mesh filename="package://duckietown_description/meshes/camera.dae" scale="4.0 4.0 4.0"/>
+            </geometry>
+            <origin xyz="0.0 0 0" rpy="0 0 0"/>
+        </collision>
+    </link>
+    <!-- tag camera ditambahkan, cek pada step ke 6. Adding the Camera to the Robot -->
 </robot>

Commit message: Add some specific data

File: rosbots_description/urdf/rosbots.gazebo.xacro (robot description, xacro)
@@ -53,3 +53,52 @@
     </sensor>
   </gazebo>
+<!-- Edit rosbots.gazebo.xacro to add the camera behavior (like take image or record video) to the link, see step 6. Adding the Camera to the Robot -->
+<!-- Edit rosbots.gazebo.xacro to add the IMU sensor, see step 7. Adding the IMU Sensor to the Robot -->
+  <gazebo>
+    <plugin name="gazebo_ros_imu_controller" filename="libgazebo_ros_imu.so">
+      <!-- <robotNamespace></robotNamespace> -->
+      <topicName>imu/data</topicName>
+      <serviceName>imu/service</serviceName>
+      <bodyName>base_link</bodyName>
+      <gaussianNoise>0</gaussianNoise>
+      <rpyOffsets>0 0 0</rpyOffsets>
+      <updateRate>30.0</updateRate>
+      <alwaysOn>true</alwaysOn>
+      <gaussianNoise>0</gaussianNoise>
+    </plugin>
+  </gazebo>
+<!-- Edit rosbots.gazebo.xacro to add the IMU sensor, see step 7. Adding the IMU Sensor to the Robot -->
+<gazebo reference="wheel_left_link">
+  <mu1>1.0</mu1>
+  <mu2>1.0</mu2>
+  <kp>1000000.0</kp>
+  <kd>100.0</kd>
+  <minDepth>0.001</minDepth>
+  <maxVel>1.0</maxVel>
+</gazebo>
+<gazebo reference="wheel_right_link">
+  <mu1>1.0</mu1>
+  <mu2>1.0</mu2>
+  <kp>1000000.0</kp>
+  <kd>100.0</kd>
+  <minDepth>0.001</minDepth>
+  <maxVel>1.0</maxVel>
+</gazebo>
+<gazebo reference="base_link">
+  <material>Gazebo/Blue</material>
+  <mu1>0.3</mu1>
+  <mu2>0.3</mu2>
+  <sensor type="contact" name="bumpers">
+    <always_on>1</always_on>
+    <update_rate>50.0</update_rate>
+    <visualize>true</visualize>
+    <contact>
+      <collision>base_footprint_collision_base_link</collision>
+    </contact>
+  </sensor>
+</gazebo>
+<gazebo reference="camera_link">
+  <mu1>0.2</mu1>
+  <mu2>0.2</mu2>
+</gazebo>
 </robot>
